Commit message: correcciones

File: example_2/description/ros2_control/diffbot.ros2_control.xacro (robot description, xacro)
@@ -1,22 +1,23 @@
 <?xml version="1.0"?>
 <robot xmlns:xacro="http://www.ros.org/wiki/xacro">
-  <xacro:macro name="diffbot_ros2_control" params="name prefix ">
+  <xacro:macro name="diffbot_ros2_control" params="name prefix">
+  <!-- <xacro:macro name="diffbot_ros2_control" params="name prefix use_mock_hardware">   -->
     <ros2_control name="${name}" type="system">
       <hardware>
         <plugin>ros2_control_demo_example_2/DiffBotSystemHardware</plugin>
         <param name="left_wheel_name">left_wheel_joint</param>
-        <param name="right_wheel_name">right_wheel_name</param>
+        <param name="right_wheel_name">right_wheel_joint</param>
         <param name="loop_rate">30</param>
-        <param name="device">/dev/ttyAMA0</param>
-        <param name="baud rate">57600</param>
-        <param name="timout_ms">1000</param>
+        <param name="device">/dev/ttyACM0</param>
+        <param name="baud_rate">115200</param>
+        <param name="timeout_ms">1000</param>
         <param name="enc_counts_per_rev">3436</param>
       </hardware>
-      <joint name="$(prefix)left_wheel_joint">
+      <joint name="${prefix}left_wheel_joint">
          <command_interface name="velocity"/>
          <state_interface name="position"/>
          <state_interface name="velocity"/>
       </joint>
-      <joint name="$(prefix)right_wheel_joint">
+      <joint name="${prefix}right_wheel_joint">
          <command_interface name="velocity"/>
          <state_interface name="position"/>

File: example_2/description/urdf/diffbot.urdf.xacro (robot description, xacro)
@@ -3,5 +3,5 @@
 <robot xmlns:xacro="http://www.ros.org/wiki/xacro" name="diffdrive_robot">
   <xacro:arg name="prefix" default="" />
-  <xacro:arg name="use_mock_hardware" default="false" />
+  <!-- <xacro:arg name="use_mock_hardware" default="false" />  -->
   <xacro:include filename="$(find ros2_control_demo_description)/diffbot/urdf/diffbot_description.urdf.xacro" />
   <!-- Import Rviz colors -->
@@ -10,5 +10,5 @@
   <xacro:include filename="$(find ros2_control_demo_example_2)/ros2_control/diffbot.ros2_control.xacro" />
   <xacro:diffbot prefix="$(arg prefix)" />
-  <xacro:diffbot_ros2_control
-    name="DiffBot" prefix="$(arg prefix)" use_mock_hardware="$(arg use_mock_hardware)"/>
+  <xacro:diffbot_ros2_control name="DiffBot" prefix="$(arg prefix)"/>
+  <!-- name="DiffBot" prefix="$(arg prefix)" use_mock_hardware="$(arg use_mock_hardware)"/>   -->
 </robot>
