Commit message: everything working

File: example_2/description/urdf/diffbot.urdf.xacro (robot description, xacro)
@@ -9,4 +9,5 @@
   <!-- Import diffbot ros2_control description -->
   <xacro:include filename="$(find ros2_control_demo_example_2)/ros2_control/diffbot.ros2_control.xacro" />
+  <!-- <xacro:include filename="$(find ros2_control_demo_descripton)/diffbot/urdf/lidar.xacro" /> -->
   <xacro:diffbot prefix="$(arg prefix)" />
   <xacro:diffbot_ros2_control name="DiffBot" prefix="$(arg prefix)"/>

File: ros2_control_demo_description/diffbot/urdf/diffbot_description.urdf.xacro (robot description, xacro)
@@ -22,4 +22,12 @@
       </geometry>
     </collision>
+    <!-- BASE_FOOTPRINT LINK -->
+    <!-- <joint name="base_footprint_joint" type="fixed">
+      <parent link="${prefix}base_link"/>
+      <child link="${prefix}base_footprint"/>
+      <origin xyz="0 0 0" rcpy="0 0 0"/>
+    </joint>
+    <link name ="{prefix}base_footprint">
+    </link> -->
     <visual>
       <origin xyz="0 0 ${base_height/2}" rpy="0 0 0"/>
@@ -149,5 +157,5 @@
           <sphere radius="${caster_wheel_radius}"/>
         </geometry>
-        <material name="white"/>
+        <material name="blue"/>
       </visual>
       <inertial>
@@ -160,4 +168,22 @@
         </inertial>
       </link>
+    <!-- <joint name="laser_joint" type="fixed">
+        <parent link="chassis"/>
+        <child link="laser_frame"/>
+        <origin xyz="0.1 0 0.175" rpy="0 0 0"/>
+    </joint>
+    <link name="laser_frame">
+        <visual>
+            <geometry>
+                <cylinder length="0.04" radius="0.05"/>
+            </geometry>
+            <material name="red"/>
+        </visual>
+        <collision>
+            <geometry>
+                <cylinder radius="0.05" length="0.04"/>
+            </geometry>
+        </collision>
+    </link> -->
   </xacro:macro>
 </robot>
