Commit message: stable

File: ros2_control_demo_description/diffbot/urdf/diffbot_description.urdf.xacro (robot description, xacro)
@@ -22,6 +22,21 @@
       </geometry>
     </collision>
+  <!-- Chasis  -->
+  <joint name="chassis_joint" type="fixed">
+    <parent link="base_link"/>
+    <child link="chassis"/>
+    <origin xyz="-0.1 0 0"/>
+  </joint>
+  <link name="chassis">
+      <visual>
+          <origin xyz="0.15 0 0.075" rpy="0 0 0"/>
+          <geometry>
+              <box size="0.3 0.3 0.15"/>
+          </geometry>
+          <material name="white"/>
+      </visual>
+  </link>
     <!-- BASE_FOOTPRINT LINK -->
-    <!-- <joint name="base_footprint_joint" type="fixed">
+    <joint name="base_footprint_joint" type="fixed">
       <parent link="${prefix}base_link"/>
       <child link="${prefix}base_footprint"/>
@@ -29,5 +44,5 @@
     </joint>
     <link name ="{prefix}base_footprint">
-    </link> -->
+    </link>
     <visual>
       <origin xyz="0 0 ${base_height/2}" rpy="0 0 0"/>
@@ -168,6 +183,6 @@
         </inertial>
       </link>
-    <!-- <joint name="laser_joint" type="fixed">
-        <parent link="chassis"/>
+    <joint name="laser_joint" type="fixed">
+        <parent link="${prefix}base_link"/>
         <child link="laser_frame"/>
         <origin xyz="0.1 0 0.175" rpy="0 0 0"/>
@@ -185,5 +200,5 @@
             </geometry>
         </collision>
-    </link> -->
+    </link>
   </xacro:macro>
 </robot>
