Commit message: small changes

File: ros2_control_demo_description/diffbot/urdf/completo.xacro (robot description, xacro)
@@ -42,21 +42,23 @@
       <origin xyz="-0.1 0 0"/>
     </joint>
-    <link name="laser_frame">
+    <!-- BASE_FOOTPRINT LINK -->
+    <link name ="{prefix}base_footprint">
       <visual>
+        <origin xyz="0 0 ${base_height/2}" rpy="0 0 0"/>
         <geometry>
-          <cylinder length="0.04" radius="0.05"/>
+          <box size="${base_width} ${base_length} ${base_height}"/>
         </geometry>
-        <material name="red"/>
+        <material name="orange"/>
       </visual>
-      <collision>
-        <geometry>
-          <cylinder radius="0.05" length="0.04"/>
-        </geometry>
-      </collision>
+      <inertial>
+        <origin xyz="0 0 0" rpy="0 0 0"/>
+        <mass value="${base_mass}"/>
+        <inertia ixx="${base_mass / 12.0 * (base_length*base_length + base_height*base_height)}" ixy="0.0" ixz="0.0" iyy="${base_mass / 12.0 * (base_height*base_height + base_width*base_width)}" iyz="0.0" izz="${base_mass / 12.0 * (base_width*base_width + base_length*base_length)}"/>
+      </inertial>
     </link>
-    <joint name="laser_joint" type="fixed">
-      <parent link="${prefix}chassis"/>
-      <child link="laser_frame"/>
-      <origin xyz="0.1 0 0.175" rpy="0 0 0"/>
+    <joint name="base_footprint_joint" type="fixed">
+      <parent link="${prefix}base_link"/>
+      <child link="${prefix}base_footprint"/>
+      <origin xyz="0 0 0" rcpy="0 0 0"/>
     </joint>
     <!-- left wheel Link -->
@@ -170,4 +172,22 @@
       <origin xyz="${base_width/2 - caster_wheel_radius} 0 ${z_offset}" rpy="0 0 0"/>
     </joint>
+    <link name="laser_frame">
+      <visual>
+        <geometry>
+          <cylinder length="0.04" radius="0.05"/>
+        </geometry>
+        <material name="red"/>
+      </visual>
+      <collision>
+        <geometry>
+          <cylinder radius="0.05" length="0.04"/>
+        </geometry>
+      </collision>
+    </link>
+    <joint name="laser_joint" type="fixed">
+      <parent link="${prefix}chassis"/>
+      <child link="laser_frame"/>
+      <origin xyz="0.1 0 0.175" rpy="0 0 0"/>
+    </joint>
   </xacro:macro>
 </robot>
